File: Schematic Diagram/ras.kicad_sch (KiCad schematic)
At the start: 2 parts

Commit message: put RC522
Parts:
- added U?: I2C_transport_LCD, symbol project:I2C_transport_LCD
Connections:
- net at RP1.3 (GPIO_2/[I2C]_SDA): now also U?. (VCC)
- net at RP1.5 (GPIO_3/[I2C]_SCL): now also U?. (VCC)
- net GND: now reaches RFID?.6 (GND)
- net GND: now also U?. (VCC)
- net +3V3: now reaches RFID?.8 (3,3V)
- new net +5V: U?. (VCC)
Other:
- moved on the sheet: RFID?

Commit message: put LED
Parts:
- removed U?: I2C_transport_LCD, symbol project:I2C_transport_LCD
- added D?: LED_RED, symbol Device:LED
- added D?: LED_GREEN, symbol Device:LED
- added D?: LED_BLUE, symbol Device:LED
- added LCD_Module?: I2C_transport_LCD, symbol project:I2C_transport_LCD
- added R? (x3): 45Ω, symbol Device:R
Connections:
- net +3V3: now also RP1.1 (+3.3V_1), RP1.17 (+3.3V_2)
- net +5V: now also RP1.2 (+5V_1), RP1.4 (+5V_2), LCD_Module?. (VCC)
- net GND: now also RP1.14 (GND_3), RP1.20 (GND_4), RP1.6 (GND_1), RP1.9 (GND_2), LCD_Module?. (VCC), R?.1, R?.1, R?.1
- net LED-RED: now reaches RP1.13 (GPIO27)
- net LED-RED: now also D?.2 (A)
- net LED-GREEN: now reaches RP1.15 (GPIO_22)
- net LED-GREEN: now also D?.2 (A)
- net LED-BLUE: now reaches RP1.16 (GPIO_23)
- net LED-BLUE: now also D?.2 (A)
- net at RP1.3 (GPIO_2/[I2C]_SDA): now also LCD_Module?. (VCC)
- net at RP1.5 (GPIO_3/[I2C]_SCL): now also LCD_Module?. (VCC)
- new net: D?.1 (K), R?.2 (x3)
Other:
- moved on the sheet: RFID?

Commit message: refactaring
Connections:
- net GND: now also RP1.25 (GND_5), RP1.30 (GND_6), RP1.34 (GND_7), RP1.39 (GND_8)
- net SPI_MOSI: now reaches RFID?.3 (MOSI), RP1.19 (GPIO_10/SPI0_MOSI)
- net SPI_MISO: now reaches RFID?.4 (MISO), RP1.21 (GPIO_9/SPI0_MISO)
- net RFID-RST: now reaches RFID?.7 (RST), RP1.22 (GPIO_25)
- net SPI_SCLK: now reaches RFID?.2 (SCK), RP1.23 (GPIO_11/SPI0_SCLK)
- net SPI_CE-RFID: now reaches RFID?.1 (SDA), RP1.24 (GPIO_8/SPI0_CE1_N)
- net I2C_SDA: now reaches LCD_Module?. (VCC), RP1.3 (GPIO_2/[I2C]_SDA)
- net I2C_SCL: now reaches LCD_Module?. (VCC), RP1.5 (GPIO_3/[I2C]_SCL)
Other:
- moved on the sheet: LCD_Module?, RFID?

Commit message: put buzzer
Parts:
- added Q?: S8050, Package_TO_SOT_THT:TO-92_Inline, symbol Transistor_BJT:S8050
- added R? (x2): Ω, symbol Device:R
Connections:
- net +5V: now also R?.2
- net GND: now also Q?.1 (E)
- net Buzzer: now reaches RP1.32 (GPIO12/PWM0)
- net Buzzer: now also R?.1
- new net: Q?.3 (C), R?.1
- new net: Q?.2 (B), R?.2
Other:
- moved on the sheet: D?, LCD_Module?, R?, RFID?, RP1

Commit message: 抵抗値変更
Parts:
- added BZ1: Buzzer, symbol Device:Buzzer
- R1, R2, R3: renamed from R?; value 45Ω -> 130Ω
- R4, R5: renamed from R?; value Ω -> 1kΩ
- gave numbers to parts that had none: 6
Connections:
- net +5V: now also BZ1.1 (-)
- net at Q1.3 (C), R5.1: now also BZ1.2 (+)
- no-connect marks 0 -> 20
Other:
- moved on the sheet: R5

Commit message: buzzer
Parts:
- added BZ?: Buzzer, symbol Device:Buzzer
- added R?: 1kΩ, symbol Device:R
Connections:
- net Buzzer: now also R?.1
- net GND: now also BZ?.2 (+)
- new net: BZ?.1 (-), R?.2
Changed lines of the file:
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@@
+    (stroke (width 0) (type default) (color 0 0 0 0))
+  )
+  (wire (pts (xy 213.36 128.27) (xy 213.36 132.08))
     (stroke (width 0) (type default) (color 0 0 0 0))
   )
@@
   )
   (wire (pts (xy 124.46 31.75) (xy 124.46 36.83))
+    (stroke (width 0) (type default) (color 0 0 0 0))
+  )
+  (wire (pts (xy 213.36 120.65) (xy 213.36 123.19))
+    (stroke (width 0) (type default) (color 0 0 0 0))
+  )
+  (wire (pts (xy 213.36 110.49) (xy 213.36 113.03))
     (stroke (width 0) (type default) (color 0 0 0 0))
   )
@@
     )
   )
+  (global_label "Buzzer" (shape input) (at 213.36 110.49 90) (fields_autoplaced)
+    (effects (font (size 1.27 1.27)) (justify left))
+    (property "シート間のリファレンス" "${INTERSHEET_REFS}" (id 0) (at 213.4394 101.7269 90)
+      (effects (font (size 1.27 1.27)) (justify left) hide)
+    )
+  )
   (global_label "LED-GREEN" (shape input) (at 80.01 115.57 0) (fields_autoplaced)
     (effects (font (size 1.27 1.27)) (justify left))
@@
     )
     (property "Datasheet" "" (id 3) (at 133.35 104.14 0)
+      (effects (font (size 1.27 1.27)) hide)
+    )
+    (pin "1")
+  )
+  (symbol (lib_id "Device:Buzzer") (at 215.9 125.73 0) (unit 1)
+    (in_bom yes) (on_board yes)
+    (property "Reference" "BZ?" (id 0) (at 219.71 124.4599 0)
+      (effects (font (size 1.27 1.27)) (justify left))
+    )
+    (property "Value" "Buzzer" (id 1) (at 219.71 126.9999 0)
+      (effects (font (size 1.27 1.27)) (justify left))
+    )
+    (property "Footprint" "" (id 2) (at 215.265 123.19 90)
+      (effects (font (size 1.27 1.27)) hide)
+    )
+    (property "Datasheet" "~" (id 3) (at 215.265 123.19 90)
+      (effects (font (size 1.27 1.27)) hide)
+    )
+    (pin "1")
+    (pin "2")
+  )
+  (symbol (lib_id "power:GND") (at 213.36 132.08 0) (unit 1)
+    (in_bom yes) (on_board yes) (fields_autoplaced)
+    (property "Reference" "#PWR?" (id 0) (at 213.36 138.43 0)
+      (effects (font (size 1.27 1.27)) hide)
+    )
+    (property "Value" "GND" (id 1) (at 213.36 137.16 0))
+    (property "Footprint" "" (id 2) (at 213.36 132.08 0)
+      (effects (font (size 1.27 1.27)) hide)
+    )
+    (property "Datasheet" "" (id 3) (at 213.36 132.08 0)
       (effects (font (size 1.27 1.27)) hide)
     )
@@
     (pin "3")
   )
+  (symbol (lib_id "Device:R") (at 213.36 116.84 0) (unit 1)
+    (in_bom yes) (on_board yes) (fields_autoplaced)
+    (property "Reference" "R?" (id 0) (at 215.9 115.5699 0)
+      (effects (font (size 1.27 1.27)) (justify left))
+    )
+    (property "Value" "1kΩ" (id 1) (at 215.9 118.1099 0)
+      (effects (font (size 1.27 1.27)) (justify left))
+    )
+    (property "Footprint" "" (id 2) (at 211.582 116.84 90)
+      (effects (font (size 1.27 1.27)) hide)
+    )
+    (property "Datasheet" "~" (id 3) (at 213.36 116.84 0)
+      (effects (font (size 1.27 1.27)) hide)
+    )
+    (pin "1")
+    (pin "2")
+  )
   (symbol (lib_id "Device:LED") (at 73.66 128.27 0) (unit 1)
     (in_bom yes) (on_board yes) (fields_autoplaced)
@@
       (reference "#PWR0111") (unit 1) (value "GND") (footprint "")
     )
+    (path "/31e494ea-4f3e-4a89-8b23-d516a4ba1b7e"
+      (reference "#PWR?") (unit 1) (value "GND") (footprint "")
+    )
     (path "/47bac56f-4f0f-44af-9cf2-8d596f7cfcf6"
       (reference "BZ1") (unit 1) (value "Buzzer") (footprint "")
     )
+    (path "/2b6301a3-5467-4fc1-bb31-50e77447df18"
+      (reference "BZ?") (unit 1) (value "Buzzer") (footprint "")
+    )
     (path "/0728d564-ee5a-4755-9671-05558f596eca"
       (reference "D1") (unit 1) (value "LED_RED") (footprint "")
@@
       (reference "R5") (unit 1) (value "1kΩ") (footprint "")
     )
+    (path "/80799c2a-76f2-481e-9d8a-e460f9a28646"
+      (reference "R?") (unit 1) (value "1kΩ") (footprint "")
+    )
     (path "/673db0f5-6dcd-4be2-a2b8-55ffc79734bd"

Commit message: update Schematic Diagram
Parts:
- gave numbers to parts that had none: 2
Changed lines of the file:
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@@
   (symbol (lib_id "Device:Buzzer") (at 215.9 125.73 0) (unit 1)
     (in_bom yes) (on_board yes)
-    (property "Reference" "BZ?" (id 0) (at 219.71 124.4599 0)
+    (property "Reference" "BZ2" (id 0) (at 219.71 124.4599 0)
       (effects (font (size 1.27 1.27)) (justify left))
     )
@@
   (symbol (lib_id "power:GND") (at 213.36 132.08 0) (unit 1)
     (in_bom yes) (on_board yes) (fields_autoplaced)
-    (property "Reference" "#PWR?" (id 0) (at 213.36 138.43 0)
+    (property "Reference" "#PWR01" (id 0) (at 213.36 138.43 0)
       (effects (font (size 1.27 1.27)) hide)
     )
@@
   (symbol (lib_id "Device:R") (at 213.36 116.84 0) (unit 1)
     (in_bom yes) (on_board yes) (fields_autoplaced)
-    (property "Reference" "R?" (id 0) (at 215.9 115.5699 0)
+    (property "Reference" "R6" (id 0) (at 215.9 115.5699 0)
       (effects (font (size 1.27 1.27)) (justify left))
     )
@@
   )
   (symbol_instances
+    (path "/31e494ea-4f3e-4a89-8b23-d516a4ba1b7e"
+      (reference "#PWR01") (unit 1) (value "GND") (footprint "")
+    )
     (path "/9904f989-d762-428d-9557-3ffdcf9e2443"
       (reference "#PWR0101") (unit 1) (value "GND") (footprint "")
@@
       (reference "#PWR0111") (unit 1) (value "GND") (footprint "")
     )
-    (path "/31e494ea-4f3e-4a89-8b23-d516a4ba1b7e"
-      (reference "#PWR?") (unit 1) (value "GND") (footprint "")
-    )
     (path "/47bac56f-4f0f-44af-9cf2-8d596f7cfcf6"
       (reference "BZ1") (unit 1) (value "Buzzer") (footprint "")
     )
     (path "/2b6301a3-5467-4fc1-bb31-50e77447df18"
-      (reference "BZ?") (unit 1) (value "Buzzer") (footprint "")
+      (reference "BZ2") (unit 1) (value "Buzzer") (footprint "")
     )
     (path "/0728d564-ee5a-4755-9671-05558f596eca"
@@
     )
     (path "/80799c2a-76f2-481e-9d8a-e460f9a28646"
-      (reference "R?") (unit 1) (value "1kΩ") (footprint "")
+      (reference "R6") (unit 1) (value "1kΩ") (footprint "")
     )
     (path "/673db0f5-6dcd-4be2-a2b8-55ffc79734bd"

Commit message: add shutdown switch close #6
Parts:
- added SW2: SW_DPST_x2, symbol Switch:SW_DPST_x2
Connections:
- net GND: now also SW2.1 (A)
- net at RP1.7 (GPIO_4/GPCLK0): now also SW2.2 (B)
- no-connect marks 20 -> 19
